File: hardware/7segement4digits1badidea-mk-1.brd (EAGLE design)
At the start: 60 x 20 mm, 18 parts, among them U1 ATTINY4313

Commit message: ADD ALL THE VERSIONS
Parts:
- removed AVRISP0: AVR_SPI_PRG_6AVR-JST-PTH-RA-I2C, A_butts:AVR-JST-6-PTH-RA-I2C
- removed U$3, U$4: (no value), A_butts:COW_SMALL
- added AVRISP1: AVR_SPI_PRG_6PTH_INLINE_I2C, A_butts:AVR_ISP_INLINE_PTH_I2C
- C3: value (none) -> 10uF; device A_butts:E2-4 -> A_butts:C025-024X044
- moved AVRISP 55.0 mm to (2.50, 10.0), turned to 90 degrees
- moved U$5 8.56 mm to (45.0, 2.20)
- moved U$6 8.56 mm to (45.0, 2.20)
- moved C2 8.50 mm to (39.0, 8.70)
- moved C3 8.07 mm to (7.00, 6.00), flipped to the top, turned to 270 degrees
- moved R1 1.00 mm to (11.0, 10.0)
Connections:
- net GND: now also C3.2; no longer AVRISP0.GND, C3.-
- net MISO: no longer AVRISP0.MISO
- net MOSI/SDA: no longer AVRISP0.MOSI/SDA
- net RESET: no longer AVRISP0.RESET
- net SCK/SCL: no longer AVRISP0.SCK
- net VCC: now also C3.1; no longer AVRISP0.VCC, C3.+
Routing:
- net VCC: track 74.7 -> 39.6 mm
- net MOSI/SDA: track 41.7 -> 19.8 mm
- net RESET: track 52.3 -> 31.2 mm
- net MISO: track 43.5 -> 22.5 mm
- net SCK/SCL: track 44.5 -> 25.5 mm
- net GND: track 3.40 -> 6.10 mm
Other:
- board text removed: "_ _ \\_(^-^)_/ uF"
