File: hardware/7segement4minidigits1badidea-mk-2.sch (EAGLE design)
At the start: 12 parts, among them U1 ATTINY4313

Commit message: ADD ALL THE VERSIONS
Parts:
- removed AVRISP: AVR_SPI_PRG_6PTH, A_butts:AVR_SPI_PRG_6PTH
- removed AVRISP1: AVR_SPI_PRG_6PTH_INLINE_I2C, A_butts:AVR_SPI_PRG_6PTH_INLINE_I2C
- removed C3: 10uF, A_butts:CAPACITOR-CERAMIC025-024X044
- removed DISPLAY1: 7SED_4DIGIT_14MM14.2MM-CC, A_butts:7SED_4DIGIT_14MM14.2MM-CC
- removed U1: ATTINY4313, A_butts:ATTINY2313ADIP
- added BUBBLES!: (>^_^)>, A_butts:7-SEGMENT-4DIGIT-COUNTERWAT
- added IC1: MC14489BSOIC, A_butts:MC14489BSOIC
- added JP1: M05PTH, A_butts:M05PTH
- C1: value 0.1uF -> 1uF; device A_butts:CAPACITOR-CERAMIC025-024X044 -> A_butts:CAPACITOR-CERAMICC0805
- C2: value 1uF -> 0.1uF; device A_butts:CAPACITOR-CERAMIC025-024X044 -> A_butts:CAPACITOR-CERAMICC0603
- R1: value 10k -> 2.2k; device A_butts:RESISTORPTH-AXIAL-7.68MM -> A_butts:RESISTORR0603
Connections:
- removed net A: DISPLAY1.A, U1.PD4
- removed net B: DISPLAY1.B, U1.PA1
- removed net C: DISPLAY1.C, U1.PB2
- removed net COLON_K: DISPLAY1.COLON_K, U1.PD1
- removed net D: DISPLAY1.D, U1.PB0
- removed net DIG1: DISPLAY1.DIG1, U1.PD5
- removed net DIG2: DISPLAY1.DIG2, U1.PD2
- removed net DIG3: DISPLAY1.DIG3, U1.PA0
- removed net DIG4: DISPLAY1.DIG4, U1.PB4
- removed net DP: DISPLAY1.DP, U1.PB1
- removed net E: DISPLAY1.E, U1.PD6
- removed net F: DISPLAY1.F, U1.PD3
- removed net G: DISPLAY1.G, U1.PB3
- removed net MISO: AVRISP.MISO, U1.PB6
- removed net MOSI/SDA: AVRISP.MOSI, U1.PB5
- removed net RESET: AVRISP.RST, R1.2, U1.PA2/!RESET
- removed net SCK/SCL: AVRISP.SCK, U1.PB7
- new net !EN: IC1.!EN, JP1.5
- new net CLOCK: IC1.CLK, JP1.4
- new net DATA: IC1.DIN, JP1.3
- new net N$1: BUBBLES!.A, IC1.A
- new net N$10: BUBBLES!.D2, IC1.DIGIT2
- new net N$11: BUBBLES!.D3, IC1.DIGIT3
- new net N$12: BUBBLES!.D4, IC1.DIGIT4
- new net N$15: IC1.I_SET, R1.2
- new net N$2: BUBBLES!.B, IC1.B
- new net N$3: BUBBLES!.C, IC1.C
- new net N$4: BUBBLES!.D, IC1.D
- new net N$5: BUBBLES!.E, IC1.E
- new net N$6: BUBBLES!.F, IC1.F
- new net N$7: BUBBLES!.G, IC1.G
- new net N$8: BUBBLES!.DP, IC1.DP
- new net N$9: BUBBLES!.D1, IC1.DIGIT1
- net GND: now also IC1.GND, JP1.1, R1.1; no longer AVRISP.GND, C3.2, U1.GND
- net VCC: now also IC1.VCC, JP1.2; no longer AVRISP.VCC, C3.1, DISPLAY1.COLON_A, R1.1, U1.VCC
Other:
- moved on the sheet: C1, C2, R1
