File: hardware/7segement4minidigits1badidea-mk-3.sch (EAGLE design)
At the start: 12 parts, among them U1 ATTINY4313

Commit message: ADD ALL THE VERSIONS
Parts:
- removed AVRISP: AVR_SPI_PRG_6PTH, A_butts:AVR_SPI_PRG_6PTH
- removed AVRISP1: AVR_SPI_PRG_6PTH_INLINE_I2C, A_butts:AVR_SPI_PRG_6PTH_INLINE_I2C
- removed C3: 10uF, A_butts:CAPACITOR-CERAMIC025-024X044
- removed DISPLAY1: 7SED_4DIGIT_14MM14.2MM-CC, A_butts:7SED_4DIGIT_14MM14.2MM-CC
- removed H3, H4: HOLE#2, A_butts:HOLE#2
- added BUBBLES!: (>^_^)>, A_butts:7-SEGMENT-4DIGIT-COUNTERWAT
- added J1: AVR_SPI_PRG_6PTH_INLINE_I2C, A_butts:AVR_SPI_PRG_6PTH_INLINE_I2C
- C1: value 0.1uF -> 1uF; device A_butts:CAPACITOR-CERAMIC025-024X044 -> A_butts:CAPACITOR-CERAMICC0805
- C2: value 1uF -> 0.1uF; device A_butts:CAPACITOR-CERAMIC025-024X044 -> A_butts:CAPACITOR-CERAMICC0603
- R1: device A_butts:RESISTORPTH-AXIAL-7.68MM -> A_butts:RESISTORR0603
- U1: value ATTINY4313 -> ATTINY2313A; device A_butts:ATTINY2313ADIP -> A_butts:ATTINY2313ASOIC
Connections:
- removed net COLON_K: DISPLAY1.COLON_K, U1.PD1
- net A: now also BUBBLES!.A, U1.PD0; no longer DISPLAY1.A, U1.PD4
- net B: now also BUBBLES!.B, U1.PD1; no longer DISPLAY1.B, U1.PA1
- net C: now also BUBBLES!.C, U1.PD6; no longer DISPLAY1.C, U1.PB2
- net D: now also BUBBLES!.D, U1.PD4; no longer DISPLAY1.D, U1.PB0
- net DIG1: now also BUBBLES!.D1, U1.PB3; no longer DISPLAY1.DIG1, U1.PD5
- net DIG2: now also BUBBLES!.D2, U1.PB2; no longer DISPLAY1.DIG2, U1.PD2
- net DIG3: now also BUBBLES!.D3, U1.PB1; no longer DISPLAY1.DIG3, U1.PA0
- net DIG4: now also BUBBLES!.D4, U1.PB0; no longer DISPLAY1.DIG4, U1.PB4
- net DP: now also BUBBLES!.DP, U1.PB4; no longer DISPLAY1.DP, U1.PB1
- net E: now also BUBBLES!.E, U1.PD2; no longer DISPLAY1.E, U1.PD6
- net F: now also BUBBLES!.F; no longer DISPLAY1.F
- net G: now also BUBBLES!.G, U1.PD5; no longer DISPLAY1.G, U1.PB3
- net GND: now also J1.GND; no longer AVRISP.GND, C3.2
- net MISO: now also J1.MISO; no longer AVRISP.MISO
- net MOSI/SDA: now also J1.MOSI; no longer AVRISP.MOSI
- net RESET: now also J1.RST; no longer AVRISP.RST
- net SCK/SCL: now also J1.SCK; no longer AVRISP.SCK
- net VCC: now also J1.VCC; no longer AVRISP.VCC, C3.1, DISPLAY1.COLON_A
Other:
- moved on the sheet: C1, C2, R1, U1
