File: hardware/7segement2digits1badidea-mk-4.2.brd (EAGLE design)
At the start: 30 x 30 mm, 11 parts, among them Q1 2N7000, U1 ATTINY84, U2 7SEG_2DIG19MM_SMT

Commit message: more dicking about
Parts:
- removed S1: SWITCH-SPDTPTH-RA-2.54MM, A_butts:SPDT-RA-2.54MM
- removed S2: SPST-NO-TACTSMD-TINY, A_butts:TACTILE-SWITCH-SMD
- added ON/OFF: SWITCH-SPDTPTH-RA-2.54MM, A_butts:SPDT-RA-2.54MM
- added RESET: SPST-NO-TACT3MM-RA, A_butts:TACTILE-PTH-SIDE
- U2: value 7SEG_2DIG19MM_SMT -> 7SEG_2DIG19MM_SMT_LESSSILK; device A_butts:7SEG_2DIG_19MM_SMT -> A_butts:7SEG_2DIG_19MM_SMT_LESSSILK
- moved C1 19.5 mm to (21.0, 5.50), turned to 0 degrees
- moved R2 19.1 mm to (9.00, 22.5), flipped to the bottom, turned to 90 degrees
- moved AVRISP 19.0 mm to (25.0, 24.0), flipped to the bottom, turned to 180 degrees
- moved R1 17.8 mm to (21.0, 18.5), turned to 180 degrees
- moved U1 14.3 mm to (21.0, 12.0), turned to 90 degrees
- moved Q1 12.1 mm to (13.0, 22.5), flipped to the bottom, turned to 90 degrees
- moved U2 6.08 mm to (21.0, 14.0), flipped to the top, turned to 90 degrees
- moved BAT 4.00 mm to (19.0, 10.5), flipped to the bottom
Connections:
- removed net DP: U1.12, U2.2
- net A: now also U1.13; no longer U1.2
- net B: now also U1.12; no longer U1.3
- net C: now also U1.2; no longer U1.13
- net D: now also U1.5; no longer U1.10
- net DIG1: now also U1.7; no longer U1.5
- net DIG2: now also U1.8; no longer U1.6
- net E: now also U1.3; no longer U1.11
- net F: now also U1.10; no longer U1.8
- net G: now also U1.6; no longer U1.9
- net GND: now also RESET.2; no longer S2.B@1, S2.B@2
- net N$3: now also ON/OFF.2; no longer S1.1
- net RESET: now also RESET.1; no longer S2.A@1, S2.A@2
- net VCC: now also ON/OFF.1; no longer S1.2
Other:
- board size 30 x 30 mm -> 36 x 28 mm
