File: hardware/7segement2digits1badidea-mk-4.2.sch (EAGLE design)
At the start: 11 parts, among them Q1 2N7000, U1 ATTINY84, U2 7SEG_2DIG19MM_SMT

Commit message: more dicking about
Parts:
- removed S1: SWITCH-SPDTPTH-RA-2.54MM, A_butts:SWITCH-SPDTPTH-RA-2.54MM
- removed S2: SPST-NO-TACTSMD-TINY, A_butts:SPST-NO-TACTSMD-TINY
- added ON/OFF: SWITCH-SPDTPTH-RA-2.54MM, A_butts:SWITCH-SPDTPTH-RA-2.54MM
- added RESET: SPST-NO-TACT3MM-RA, A_butts:SPST-NO-TACT3MM-RA
- U2: value 7SEG_2DIG19MM_SMT -> 7SEG_2DIG19MM_SMT_LESSSILK; device A_butts:7SEG_2DIG19MM_SMT -> A_butts:7SEG_2DIG19MM_SMT_LESSSILK
Connections:
- removed net DP: U1.(PCINT1/AIN0/ADC1)PA1, U2.DP
- net A: now also U1.(PCINT0/AREF/ADC0)PA0; no longer U1.(PCINT8/XTAL1/CLKI)PB0
- net B: now also U1.(PCINT1/AIN0/ADC1)PA1; no longer U1.(PCINT9/XTAL2)PB1
- net C: now also U1.(PCINT8/XTAL1/CLKI)PB0; no longer U1.(PCINT0/AREF/ADC0)PA0
- net D: now also U1.(PCINT10/INT0/OC0A/CKOUT)PB2; no longer U1.(PCINT3/T0/ADC3)PA3
- net DIG1: now also U1.(PCINT6/OC1A/SDA/MOSI/ADC6)PA6; no longer U1.(PCINT10/INT0/OC0A/CKOUT)PB2
- net DIG2: now also U1.(PCINT5/OC1B/MISO/DO/ADC5)PA5; no longer U1.(PCINT7/ICP/OC0B/ADC7)PA7
- net E: now also U1.(PCINT9/XTAL2)PB1; no longer U1.(PCINT2/AIN1/ADC2)PA2
- net F: now also U1.(PCINT3/T0/ADC3)PA3; no longer U1.(PCINT5/OC1B/MISO/DO/ADC5)PA5
- net G: now also U1.(PCINT7/ICP/OC0B/ADC7)PA7; no longer U1.(PCINT4/T1/SCL/USCK/ADC4)PA4
- net GND: now also RESET.2; no longer S2.2
- net N$3: now also ON/OFF.COM; no longer S1.NC
- net RESET: now also RESET.1; no longer S2.1
- net VCC: now also ON/OFF.NC; no longer S1.COM
