File: hardware/7segement2digits1badidea-mk-4.3.brd (EAGLE design)
At the start: 31.5 x 28 mm, 11 parts, among them Q1 2N7000, U1 ATTINY84, U2 7SEG_2DIG19MM_SMT_LESSSILK

Commit message: twaddle
Parts:
- removed Q1: 2N7000, A_butts:SOT23
- removed R2: 10k, A_butts:R0805
- removed RESET: SPST-NO-TACTSMD-TINY, A_butts:TACTILE-SWITCH-SMD
- moved R1 11.3 mm to (25.5, 13.5), flipped to the top, turned to 270 degrees
- moved C1 9.30 mm to (15.5, 8.50), turned to 0 degrees
- moved AVRISP 1.45 mm to (30.6, 12.9), flipped to the bottom, turned to 90 degrees
- moved U1 1.12 mm to (15.5, 15.0), turned to 90 degrees
- moved U2 0.75 mm to (15.8, 14.0)
Connections:
- removed net N$1: Q1.1, R2.1
- removed net N$2: BAT1.BOTTOM, Q1.3
- net A: no longer U1.13
- net B: no longer U1.12
- net C: no longer U1.2
- net D: no longer U1.5
- net DIG1: now also U1.6; no longer U1.7
- net DIG2: now also U1.5; no longer U1.8
- net E: no longer U1.3
- net F: no longer U1.10
- net G: no longer U1.6
- net GND: now also BAT1.BOTTOM; no longer Q1.2, RESET.B@1, RESET.B@2
- net RESET: no longer RESET.A@1, RESET.A@2
- net VCC: no longer R2.2
Routing:
- added copper zone on layer 16, net GND
Other:
- board size 31.5 x 28 mm -> 37 x 28 mm
