File: hardware/7segement2digits1badidea-mk-4.3.sch (EAGLE design)
At the start: 11 parts, among them Q1 2N7000, U1 ATTINY84, U2 7SEG_2DIG19MM_SMT_LESSSILK

Commit message: twaddle
Parts:
- removed Q1: 2N7000, A_butts:MOSFET-NCHANNELBSS123LT1G
- removed R2: 10k, A_butts:RESISTORR0805
- removed RESET: SPST-NO-TACTSMD-TINY, A_butts:SPST-NO-TACTSMD-TINY
Connections:
- removed net N$1: Q1.G, R2.1
- removed net N$2: BAT1.-, Q1.D
- net A: no longer U1.(PCINT0/AREF/ADC0)PA0
- net B: no longer U1.(PCINT1/AIN0/ADC1)PA1
- net C: no longer U1.(PCINT8/XTAL1/CLKI)PB0
- net D: no longer U1.(PCINT10/INT0/OC0A/CKOUT)PB2
- net DIG1: now also U1.(PCINT7/ICP/OC0B/ADC7)PA7; no longer U1.(PCINT6/OC1A/SDA/MOSI/ADC6)PA6
- net DIG2: now also U1.(PCINT10/INT0/OC0A/CKOUT)PB2; no longer U1.(PCINT5/OC1B/MISO/DO/ADC5)PA5
- net E: no longer U1.(PCINT9/XTAL2)PB1
- net F: no longer U1.(PCINT3/T0/ADC3)PA3
- net G: no longer U1.(PCINT7/ICP/OC0B/ADC7)PA7
- net GND: now also BAT1.-; no longer Q1.S, RESET.2
- net RESET: no longer RESET.1
- net VCC: no longer R2.2
Other:
- moved on the sheet: BAT1
