File: hardware/7segement2digits1badidea-mk-5.1.brd (EAGLE design)
At the start: 31.5 x 28 mm, 10 parts, among them Q1 IRLML2502, U1 ATTINY84, U2 7SEG_2DIG19MM_SMT_LESSSILK

Commit message: wonderboard take me away from here
Parts:
- removed AVRISP: AVR_SPI_PRG_6AVR-JST-PTH-RA-I2C, A_butts:AVR-JST-6-PTH-RA-I2C
- removed Q1: IRLML2502, A_butts:SOT23
- removed R2: 10k, A_butts:R0805
- moved C1 14.0 mm to (23.0, 14.0), turned to 90 degrees
- moved R1 9.22 mm to (23.0, 19.0), turned to 0 degrees
- turned U1 to 180 degrees
Connections:
- removed net MOSI: AVRISP.MOSI/SDA
- removed net N$2: BAT1.BOTTOM, Q1.3
- removed net N$3: Q1.1, R2.1
- removed net SCK: AVRISP.SCK
- net A: now also U1.8
- net B: now also U1.7
- net C: now also U1.10, U1.9; no longer U1.2
- net D: now also U1.13
- net DIG1: now also U1.6
- net DIG2: now also U1.5; no longer AVRISP.MISO
- net DP: now also U1.11
- net E: now also U1.12; no longer U1.3
- net F: now also U1.3
- net G: now also U1.2
- net GND: now also BAT1.BOTTOM; no longer AVRISP.GND, Q1.2
- net RESET: no longer AVRISP.RESET
- net VCC: no longer AVRISP.VCC, R2.2
Changed lines of the file:
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@@
 </autorouter>
 <elements>
-<element name="U1" library="A_butts" package="SO14" value="ATTINY84" x="16" y="14"/>
-<element name="C1" library="A_butts" package="C0805" value="0.1uF" x="9" y="14" rot="R270"/>
+<element name="U1" library="A_butts" package="SO14" value="ATTINY84" x="16" y="14" rot="R180"/>
+<element name="C1" library="A_butts" package="C0805" value="0.1uF" x="23" y="14" rot="R90"/>
 <element name="U2" library="A_butts" package="7SEG_2DIG_19MM_SMT_LESSSILK" value="7SEG_2DIG19MM_SMT_LESSSILK" x="15.75" y="14" smashed="yes"/>
-<element name="AVRISP" library="A_butts" package="AVR-JST-6-PTH-RA-I2C" value="AVR_SPI_PRG_6AVR-JST-PTH-RA-I2C" x="29.5" y="14" smashed="yes" rot="MR90">
-<attribute name="NAME" x="29" y="5.75" size="0.7" layer="26" font="vector" ratio="12" rot="MR180" align="bottom-center"/>
-</element>
-<element name="R1" library="A_butts" package="R0805" value="10k" x="25" y="10" rot="R90"/>
+<element name="R1" library="A_butts" package="R0805" value="10k" x="23" y="19"/>
 <element name="FRAME1" library="A_butts" package="DUMMY" value="FRAME-LETTERNO_PACKAGE" x="0" y="-0.5">
 <attribute name="VERSION" value="v01" x="0" y="-0.5" size="0.5" layer="27" ratio="12" display="off"/>
@@
 <attribute name="VALUE" x="13.5" y="-3" size="0.8" layer="28" font="vector" ratio="12" rot="MR0" align="top-center"/>
 </element>
-<element name="R2" library="A_butts" package="R0805" value="10k" x="9" y="24" smashed="yes" rot="MR270">
-<attribute name="NAME" x="9" y="26" size="0.7" layer="26" font="vector" ratio="12" rot="MR0" align="bottom-center"/>
-<attribute name="VALUE" x="9" y="22" size="0.6" layer="28" font="vector" ratio="12" rot="MR0" align="top-center"/>
-</element>
 <element name="POWER" library="A_butts" package="SPDT-RA-2.54MM" value="SWITCH-SPDTPTH-RA-2.54MM" x="29" y="25.37" rot="R180"/>
-<element name="Q1" library="A_butts" package="SOT23" value="IRLML2502" x="13.5" y="23.5" smashed="yes" rot="MR180">
-<attribute name="NAME" x="13.5" y="25.5" size="0.7" layer="26" font="vector" ratio="12" rot="MR0" align="bottom-center"/>
-<attribute name="VALUE" x="13.5" y="21.5" size="0.6" layer="28" font="vector" ratio="12" rot="MR0" align="top-center"/>
-</element>
 </elements>
 <signals>
 <signal name="VCC">
-<contactref element="AVRISP" pad="VCC"/>
 <contactref element="U1" pad="1"/>
 <contactref element="C1" pad="2"/>
 <contactref element="R1" pad="2"/>
-<contactref element="R2" pad="2"/>
 <contactref element="POWER" pad="2"/>
-<wire x1="29.5" y1="19" x2="26.46" y2="25.37" width="0" layer="19" extent="1-1"/>
-<wire x1="25" y1="10.95" x2="29.5" y2="19" width="0" layer="19" extent="1-1"/>
-<wire x1="12.19" y1="11.2" x2="25" y2="10.95" width="0" layer="19" extent="1-1"/>
-<wire x1="9" y1="13.05" x2="12.19" y2="11.2" width="0" layer="19" extent="1-1"/>
-<wire x1="9" y1="23.05" x2="9" y2="13.05" width="0" layer="19" extent="1-16"/>
+<wire x1="23.95" y1="19" x2="26.46" y2="25.37" width="0" layer="19" extent="1-1"/>
+<wire x1="23" y1="14.95" x2="23.95" y2="19" width="0" layer="19" extent="1-1"/>
+<wire x1="19.81" y1="16.8" x2="23" y2="14.95" width="0" layer="19" extent="1-1"/>
 </signal>
 <signal name="GND">
-<contactref element="AVRISP" pad="GND"/>
 <contactref element="U1" pad="14"/>
 <contactref element="C1" pad="1"/>
@@
 <vertex x="-0.1" y="28.1"/>
 </polygon>
-<contactref element="Q1" pad="2"/>
 <polygon width="0.1524" layer="16">
 <vertex x="-0.1" y="-0.1"/>
@@
 <vertex x="31.6" y="-0.1"/>
 </polygon>
+<contactref element="BAT1" pad="BOTTOM"/>
+<via x="29" y="15" extent="1-16" drill="0.3302"/>
 </signal>
 <signal name="DIG1">
 <contactref element="U2" pad="8"/>
+<contactref element="U1" pad="6"/>
+<wire x1="13.46" y1="16.8" x2="15.75" y2="23.525" width="0" layer="19" extent="1-1"/>
 </signal>
 <signal name="A">
 <contactref element="U2" pad="10"/>
+<contactref element="U1" pad="8"/>
+<wire x1="12.19" y1="11.2" x2="10.67" y2="23.525" width="0" layer="19" extent="1-1"/>
 </signal>
 <signal name="RESET">
-<contactref element="AVRISP" pad="RESET"/>
 <contactref element="U1" pad="4"/>
 <contactref element="R1" pad="1"/>
-<wire x1="25" y1="9.05" x2="29.5" y2="9" width="0" layer="19" extent="1-1"/>
-<wire x1="16" y1="11.2" x2="25" y2="9.05" width="0" layer="19" extent="1-1"/>
+<wire x1="16" y1="16.8" x2="22.05" y2="19" width="0" layer="19" extent="1-1"/>
 </signal>
 <signal name="B">
 <contactref element="U2" pad="9"/>
+<contactref element="U1" pad="7"/>
+<wire x1="12.19" y1="16.8" x2="13.21" y2="23.525" width="0" layer="19" extent="1-1"/>
 </signal>
 <signal name="D">
 <contactref element="U2" pad="4"/>
+<contactref element="U1" pad="13"/>
+<wire x1="18.29" y1="4.475" x2="18.54" y2="11.2" width="0" layer="19" extent="1-1"/>
 </signal>
 <signal name="F">
 <contactref element="U2" pad="6"/>
+<contactref element="U1" pad="3"/>
+<wire x1="17.27" y1="16.8" x2="20.83" y2="23.525" width="0" layer="19" extent="1-1"/>
 </signal>
 <signal name="G">
 <contactref element="U2" pad="5"/>
+<contactref element="U1" pad="2"/>
+<wire x1="20.83" y1="4.475" x2="18.54" y2="16.8" width="0" layer="19" extent="1-1"/>
 </signal>
 <signal name="E">
 <contactref element="U2" pad="3"/>
-<contactref element="U1" pad="3"/>
-<wire x1="15.75" y1="4.475" x2="14.73" y2="11.2" width="0" layer="19" extent="1-1"/>
+<contactref element="U1" pad="12"/>
+<wire x1="15.75" y1="4.475" x2="17.27" y2="11.2" width="0" layer="19" extent="1-1"/>
 </signal>
 <signal name="C">
 <contactref element="U2" pad="1"/>
-<contactref element="U1" pad="2"/>
+<contactref element="U1" pad="10"/>
+<contactref element="U1" pad="9"/>
+<wire x1="13.46" y1="11.2" x2="14.73" y2="11.2" width="0" layer="19" extent="1-1"/>
 <wire x1="10.67" y1="4.475" x2="13.46" y2="11.2" width="0" layer="19" extent="1-1"/>
 </signal>
 <signal name="DP">
 <contactref element="U2" pad="2"/>
+<contactref element="U1" pad="11"/>
+<wire x1="13.21" y1="4.475" x2="16" y2="11.2" width="0" layer="19" extent="1-1"/>
 </signal>
 <signal name="DIG2">
 <contactref element="U2" pad="7"/>
-<contactref element="AVRISP" pad="MISO"/>
-<wire x1="29.5" y1="11" x2="18.29" y2="23.525" width="0" layer="19" extent="1-1"/>
-</signal>
-<signal name="N$2">
-<contactref element="BAT1" pad="BOTTOM"/>
-<contactref element="Q1" pad="3"/>
-<wire x1="13.5" y1="10.5" x2="13.5" y2="22.5" width="0" layer="19" extent="16-16"/>
-</signal>
-<signal name="N$3">
-<contactref element="R2" pad="1"/>
-<contactref element="Q1" pad="1"/>
-<wire x1="9" y1="24.95" x2="12.55" y2="24.5" width="0" layer="19" extent="16-16"/>
-</signal>
-<signal name="MOSI">
-<contactref element="AVRISP" pad="MOSI/SDA"/>
-</signal>
-<signal name="SCK">
-<contactref element="AVRISP" pad="SCK"/>
+<contactref element="U1" pad="5"/>
+<wire x1="14.73" y1="16.8" x2="18.29" y2="23.525" width="0" layer="19" extent="1-1"/>
 </signal>
 <signal name="N$1">
