File: hardware/7segement2digits1badidea-mk-5.1.sch (EAGLE design)
At the start: 10 parts, among them Q1 IRLML2502, U1 ATTINY84, U2 7SEG_2DIG19MM_SMT_LESSSILK

Commit message: wonderboard take me away from here
Parts:
- removed AVRISP: AVR_SPI_PRG_6AVR-JST-PTH-RA-I2C, A_butts:AVR_SPI_PRG_6AVR-JST-PTH-RA-I2C
- removed Q1: IRLML2502, A_butts:MOSFET-NCHANNELIRLML2502
- removed R2: 10k, A_butts:RESISTORR0805
Connections:
- removed net MOSI: AVRISP.MOSI
- removed net N$2: BAT1.-, Q1.D
- removed net N$3: Q1.G, R2.1
- removed net SCK: AVRISP.SCK
- net A: now also U1.(PCINT5/OC1B/MISO/DO/ADC5)PA5
- net B: now also U1.(PCINT6/OC1A/SDA/MOSI/ADC6)PA6
- net C: now also U1.(PCINT3/T0/ADC3)PA3, U1.(PCINT4/T1/SCL/USCK/ADC4)PA4; no longer U1.(PCINT8/XTAL1/CLKI)PB0
- net D: now also U1.(PCINT0/AREF/ADC0)PA0
- net DIG1: now also U1.(PCINT7/ICP/OC0B/ADC7)PA7
- net DIG2: now also U1.(PCINT10/INT0/OC0A/CKOUT)PB2; no longer AVRISP.MISO
- net DP: now also U1.(PCINT2/AIN1/ADC2)PA2
- net E: now also U1.(PCINT1/AIN0/ADC1)PA1; no longer U1.(PCINT9/XTAL2)PB1
- net F: now also U1.(PCINT9/XTAL2)PB1
- net G: now also U1.(PCINT8/XTAL1/CLKI)PB0
- net GND: now also BAT1.-; no longer AVRISP.GND, Q1.S
- net RESET: no longer AVRISP.RST
- net VCC: no longer AVRISP.VCC, R2.2
