File: hardware/7segement2digits1badidea-mk-6.0.sch (EAGLE design)
At the start: 12 parts, among them IC1 MAX7219

Commit message: whooooole bunch of designs i apparently never committed
Parts:
- removed C2: 100nF, A_butts:CAPACITOR-CERAMICC0805
- removed DISPLAY1, DISPLAY2: 7SEG_4DIGIT_COLON_APOS, A_butts:7SEG_4DIGIT_COLON_APOS
- removed IC1: MAX7219, A_butts:MAX7219SOIC-W
- removed JP1: M05PTH, A_butts:M05PTH
- removed R2, R3, R4, R5: 330R, A_butts:RESISTORR0805
- added AVRISP: AVR_SPI_PRG_62X3_SMD, A_butts:AVR_SPI_PRG_62X3_SMD
- added U1: ATTINY84, A_butts:ATTINY84
- added U2: 7SEG_2DIG14MM, A_butts:7SEG_2DIG14MM
- C1: value 1uF -> 0.1uF; device A_butts:CAPACITOR-CERAMICC0805 -> A_butts:CAPACITOR-CERAMICC0603
- R1: device A_butts:RESISTORR0805 -> A_butts:RESISTORR0603
Connections:
- removed net AP1: DISPLAY1.AP_A, R2.1
- removed net AP2: DISPLAY2.AP_A, R4.1
- removed net CL1: DISPLAY1.CL_A, R3.1
- removed net CL2: DISPLAY2.CL_A, R5.1
- removed net CLK: IC1.CLK, JP1.1
- removed net DATA: IC1.DIN, JP1.3
- removed net DIG0: DISPLAY1.DIG1, IC1.DIG0
- removed net DIG3: DISPLAY1.DIG4, IC1.DIG3
- removed net DIG4: DISPLAY2.DIG1, IC1.DIG4
- removed net DIG5: DISPLAY2.DIG2, IC1.DIG5
- removed net DIG6: DISPLAY2.DIG3, IC1.DIG6
- removed net DIG7: DISPLAY2.DIG4, IC1.DIG7
- removed net LOAD: IC1.LOAD, JP1.2
- removed net N$1: IC1.ISET, R1.1
- new net MISO: AVRISP.MISO
- new net MOSI: AVRISP.MOSI
- new net RESET: AVRISP.RST, R1.1, U1.(PCINT11/~RESET/DW)PB3
- new net SCK: AVRISP.SCK
- net A: now also U1.(PCINT5/OC1B/MISO/DO/ADC5)PA5, U2.A; no longer DISPLAY1.A, DISPLAY2.A, IC1.SEGA
- net B: now also U1.(PCINT4/T1/SCL/USCK/ADC4)PA4, U2.B; no longer DISPLAY1.B, DISPLAY2.B, IC1.SEGB
- net C: now also U1.(PCINT9/XTAL2)PB1, U2.C; no longer DISPLAY1.C, DISPLAY2.C, IC1.SEGC
- net D: now also U1.(PCINT10/INT0/OC0A/CKOUT)PB2, U2.D; no longer DISPLAY1.D, DISPLAY2.D, IC1.SEGD
- net DIG1: now also U2.DIG1; no longer DISPLAY1.DIG2, IC1.DIG1
- net DIG2: now also U1.(PCINT8/XTAL1/CLKI)PB0, U2.DIG2; no longer DISPLAY1.DIG3, IC1.DIG2
- net DP: now also U2.DP; no longer DISPLAY1.DP, DISPLAY2.DP, IC1.SEGDP
- net E: now also U1.(PCINT6/OC1A/SDA/MOSI/ADC6)PA6, U2.E; no longer DISPLAY1.E, DISPLAY2.E, IC1.SEGE
- net F: now also U1.(PCINT7/ICP/OC0B/ADC7)PA7, U2.F; no longer DISPLAY1.F, DISPLAY2.F, IC1.SEGF
- net G: now also U2.G; no longer DISPLAY1.G, DISPLAY2.G, IC1.SEGG
- net GND: now also AVRISP.GND, U1.GND; no longer C2.2, DISPLAY1.AP_K, DISPLAY1.CL_K, DISPLAY2.AP_K, DISPLAY2.CL_K, IC1.GND, IC1.GND2, JP1.4
- net VCC: now also AVRISP.VCC, U1.VCC; no longer C2.1, IC1.VCC, JP1.5, R2.2, R3.2, R4.2, R5.2
Other:
- note added: "1"
- note added: "2"
- note added: "3"
- note added: "4"
- note added: "A"
- note added: "B"
- note added: "C"
- note added: "D"
- note added: "E"
- note added: "F"
- note added: "G"
- note added: "P"
- note added: "PA0"
- note added: "PA1"
- note added: "PA2"
- note added: "PA3"
- note added: "PA4"
- note added: "PA5"
- note added: "PA6"
- note added: "PA7"
- note added: "PB0"
- note added: "PB1"
- note added: "PB2"
- moved on the sheet: C1, R1
