File: hardware/7segement4digits1badidea-max7219-smd-mk-5.0.sch (EAGLE design)
At the start: 12 parts, among them IC1 MAX7219

Commit message: whooooole bunch of designs i apparently never committed
Parts:
- removed C2: 100nF, A_butts:CAPACITOR-CERAMICC0805
- removed DISPLAY1, DISPLAY2: 7SEG_4DIGIT_COLON_APOS, A_butts:7SEG_4DIGIT_COLON_APOS
- removed R2, R3, R4, R5: 330R, A_butts:RESISTORR0805
- added DIGIT1, DIGIT2, DIGIT3, DIGIT4: 7SEG_1DIGPTH-25.4MM, A_butts:7SEG_1DIGPTH-25.4MM
- C1: value 1uF -> 100n
- FRAME1: DESIGNER (none) -> sean@yak.net; VERSION (none) -> v5.0
- JP1: value M05PTH -> M05PTH-CENTERED; device A_butts:M05PTH -> A_butts:M05PTH-CENTERED
Connections:
- removed net AP1: DISPLAY1.AP_A, R2.1
- removed net AP2: DISPLAY2.AP_A, R4.1
- removed net CL1: DISPLAY1.CL_A, R3.1
- removed net CL2: DISPLAY2.CL_A, R5.1
- removed net DIG0: DISPLAY1.DIG1, IC1.DIG0
- removed net DIG5: DISPLAY2.DIG2, IC1.DIG5
- removed net DIG6: DISPLAY2.DIG3, IC1.DIG6
- removed net DIG7: DISPLAY2.DIG4, IC1.DIG7
- new net N$2: IC1.DIG4
- new net N$3: IC1.DIG5
- new net N$4: IC1.DIG6
- new net N$5: IC1.DIG7
- net A: now also DIGIT1.A, DIGIT2.A, DIGIT3.A, DIGIT4.A; no longer DISPLAY1.A, DISPLAY2.A
- net B: now also DIGIT1.B, DIGIT2.B, DIGIT3.B, DIGIT4.B; no longer DISPLAY1.B, DISPLAY2.B
- net C: now also DIGIT1.C, DIGIT2.C, DIGIT3.C, DIGIT4.C; no longer DISPLAY1.C, DISPLAY2.C
- net D: now also DIGIT1.D, DIGIT2.D, DIGIT3.D, DIGIT4.D; no longer DISPLAY1.D, DISPLAY2.D
- net DIG1: now also DIGIT1.K1, IC1.DIG0; no longer DISPLAY1.DIG2, IC1.DIG1
- net DIG2: now also DIGIT2.K1, IC1.DIG1; no longer DISPLAY1.DIG3, IC1.DIG2
- net DIG3: now also DIGIT3.K1, IC1.DIG2; no longer DISPLAY1.DIG4, IC1.DIG3
- net DIG4: now also DIGIT4.K1, IC1.DIG3; no longer DISPLAY2.DIG1, IC1.DIG4
- net DP: now also DIGIT1.DP, DIGIT2.DP, DIGIT3.DP, DIGIT4.DP; no longer DISPLAY1.DP, DISPLAY2.DP
- net E: now also DIGIT1.E, DIGIT2.E, DIGIT3.E, DIGIT4.E; no longer DISPLAY1.E, DISPLAY2.E
- net F: now also DIGIT1.F, DIGIT2.F, DIGIT3.F, DIGIT4.F; no longer DISPLAY1.F, DISPLAY2.F
- net G: now also DIGIT1.G, DIGIT2.G, DIGIT3.G, DIGIT4.G; no longer DISPLAY1.G, DISPLAY2.G
- net GND: now also C1.2; no longer C1.1, C2.2, DISPLAY1.AP_K, DISPLAY1.CL_K, DISPLAY2.AP_K, DISPLAY2.CL_K
- net VCC: now also C1.1; no longer C1.2, C2.1, R2.2, R3.2, R4.2, R5.2
Other:
- moved on the sheet: C1
