File: hardware/7segement4digits1badidea-mk-2.0.sch (EAGLE design)
At the start: 12 parts, among them IC1 MAX7219

Commit message: whooooole bunch of designs i apparently never committed
Parts:
- removed DISPLAY1, DISPLAY2: 7SEG_4DIGIT_COLON_APOS, A_butts:7SEG_4DIGIT_COLON_APOS
- removed JP1: M05PTH, A_butts:M05PTH
- removed R2, R3, R4, R5: 330R, A_butts:RESISTORR0805
- added AVR_ISP: AVR_SPI_PRG_6PTH, A_butts:AVR_SPI_PRG_6PTH
- added DIGIT0, DIGIT1, DIGIT2, DIGIT3: 7SEG_1DIGPTH-25.4MM, A_butts:7SEG_1DIGPTH-25.4MM
- added I2C: M04-I2CPTH-0.1IN-CENTERED-FLIPPED, A_butts:M04-I2CPTH-0.1IN-CENTERED-FLIPPED
- added RESET: SPST-NO-TACT3MM-PTH-SMALL-PADS, A_butts:SPST-NO-TACT3MM-PTH-SMALL-PADS
- added UART1: M06-UARTPTH-0.1IN, A_butts:M06-UARTPTH-0.1IN
- added Y1: 16MHz, A_butts:RESONATORPTH
- C1: value 1uF -> 100n; device A_butts:CAPACITOR-CERAMICC0805 -> A_butts:CAPACITOR-CERAMIC025-024X044
- C2: value 100nF -> 100n; device A_butts:CAPACITOR-CERAMICC0805 -> A_butts:CAPACITOR-CERAMIC025-024X044
- IC1: value MAX7219 -> ATMEGA328P; device A_butts:MAX7219SOIC-W -> A_butts:ATMEGA328P_PDIP
- R1: device A_butts:RESISTORR0805 -> A_butts:RESISTORPTH-AXIAL-7.62MM
Connections:
- removed net A: DISPLAY1.A, DISPLAY2.A, IC1.SEGA
- removed net AP1: DISPLAY1.AP_A, R2.1
- removed net AP2: DISPLAY2.AP_A, R4.1
- removed net B: DISPLAY1.B, DISPLAY2.B, IC1.SEGB
- removed net C: DISPLAY1.C, DISPLAY2.C, IC1.SEGC
- removed net CL1: DISPLAY1.CL_A, R3.1
- removed net CL2: DISPLAY2.CL_A, R5.1
- removed net CLK: IC1.CLK, JP1.1
- removed net D: DISPLAY1.D, DISPLAY2.D, IC1.SEGD
- removed net DATA: IC1.DIN, JP1.3
- removed net DIG0: DISPLAY1.DIG1, IC1.DIG0
- removed net DIG1: DISPLAY1.DIG2, IC1.DIG1
- removed net DIG2: DISPLAY1.DIG3, IC1.DIG2
- removed net DIG3: DISPLAY1.DIG4, IC1.DIG3
- removed net DIG4: DISPLAY2.DIG1, IC1.DIG4
- removed net DIG5: DISPLAY2.DIG2, IC1.DIG5
- removed net DIG6: DISPLAY2.DIG3, IC1.DIG6
- removed net DIG7: DISPLAY2.DIG4, IC1.DIG7
- removed net DP: DISPLAY1.DP, DISPLAY2.DP, IC1.SEGDP
- removed net E: DISPLAY1.E, DISPLAY2.E, IC1.SEGE
- removed net F: DISPLAY1.F, DISPLAY2.F, IC1.SEGF
- removed net G: DISPLAY1.G, DISPLAY2.G, IC1.SEGG
- removed net LOAD: IC1.LOAD, JP1.2
- new net A0: DIGIT0.G, DIGIT1.G, DIGIT2.G, DIGIT3.G, IC1.PC0(ADC0)
- new net A1: DIGIT0.F, DIGIT1.F, DIGIT2.F, DIGIT3.F, IC1.PC1(ADC1)
- new net A2: DIGIT0.A, DIGIT1.A, DIGIT2.A, DIGIT3.A, IC1.PC2(ADC2)
- new net A3: DIGIT0.B, DIGIT1.B, DIGIT2.B, DIGIT3.B, IC1.PC3(ADC3)
- new net CTS: C2.2, UART1.CTS
- new net D10: DIGIT2.K2, IC1.PB2(SS/OC1B)
- new net D3: DIGIT0.DP, DIGIT1.DP, DIGIT2.DP, DIGIT3.DP, IC1.PD3(INT1)
- new net D4: DIGIT0.C, DIGIT1.C, DIGIT2.C, DIGIT3.C, IC1.PD4(XCK/T0)
- new net D5: DIGIT0.K1, IC1.PD5(T1)
- new net D6: DIGIT1.K1, IC1.PD6(AIN0)
- new net D7: DIGIT0.D, DIGIT1.D, DIGIT2.D, DIGIT3.D, IC1.PD7(AIN1)
- new net D8: DIGIT0.E, DIGIT1.E, DIGIT2.E, DIGIT3.E, IC1.PB0(ICP)
- new net D9: DIGIT3.K2, IC1.PB1(OC1A)
- new net MISO: AVR_ISP.MISO, IC1.PB4(MISO)
- new net MOSI: AVR_ISP.MOSI, IC1.PB3(MOSI/OC2)
- new net N$2: IC1.PB6(XTAL1/TOSC1), Y1.3
- new net RST: AVR_ISP.RST, C2.1, IC1.PC6(/RESET), R1.1, RESET.2
- new net RXD: IC1.PD0(RXD), UART1.TXO
- new net SCK: AVR_ISP.SCK, IC1.PB5(SCK)
- new net SCL: I2C.SCL, IC1.PC5(ADC5/SCL)
- new net SDA: I2C.SDA, IC1.PC4(ADC4/SDA)
- new net TXD: IC1.PD1(TXD), UART1.RXI
- net GND: now also AVR_ISP.GND, C1.2, I2C.GND, IC1.GND@1, IC1.GND@2, RESET.1, UART1.GND, UART1.RTS, Y1.2; no longer C1.1, C2.2, DISPLAY1.AP_K, DISPLAY1.CL_K, DISPLAY2.AP_K, DISPLAY2.CL_K, IC1.GND, IC1.GND2, JP1.4
- net N$1: now also IC1.PB7(XTAL2/TOSC2), Y1.1; no longer IC1.ISET, R1.1
- net VCC: now also AVR_ISP.VCC, C1.1, I2C.VCC, IC1.AVCC, UART1.VIN; no longer C1.2, C2.1, JP1.5, R2.2, R3.2, R4.2, R5.2
Other:
- note added: "1 = E"
- note added: "10 = G"
- note added: "2 = D"
- note added: "4 = C"
- note added: "5 = DP"
- note added: "6 = B"
- note added: "7 = A"
- note added: "9 = F"
- note added: "A"
- note added: "A0"
- note added: "A1"
- note added: "A2"
- note added: "A3"
- note added: "B"
- note added: "C"
- note added: "D"
- note added: "D10"
- note added: "D3"
- note added: "D4"
- note added: "D5"
- note added: "D6"
- note added: "D7"
- note added: "D8"
- note added: "D9"
- note added: "DP"
- note added: "E"
- note added: "F"
- note added: "G"
- moved on the sheet: C1, C2, R1
